Commit message: Tidied up, added end effector pos publisher.

File: state_publisher/urdf/simple.urdf (robot description, URDF)
Before this commit: robot Simple, 11 links, 10 joints
Links:
- added link end_effector_ref; visual sphere radius=0.02
Joints:
- added joint end_effector_ref: type fixed, parent Link_2_1, child end_effector_ref, origin xyz=0.55 0 0 rpy=0 0 0
