Commit message: Fixed robot model and rebuilt robot_config package

File: state/state_publisher/urdf/rescue.urdf (robot description, URDF)
Before this commit: robot rescue, 14 links, 13 joints
Joints:
- removed joint flipper_front
- removed joint flipper_rear
- added joint flippers_front: type revolute, parent right_belt_1, child flipper_front_right_1, origin xyz=0.454878 0.0 0.055 rpy=0 0 0, axis 0.0 0.0 0.01, limit lower=-3.316126 upper=1.570796 effort=100 velocity=100
- added joint flippers_rear: type revolute, parent right_belt_1, child flipper_rear_right_1, origin xyz=0.0 0.0 0.055 rpy=0 0 0, axis 0.0 0.0 0.01, limit lower=-1.570796 upper=3.316126 effort=100 velocity=100
- joint Rigid1: origin xyz=-0.121419 -0.029614 -0.010522 rpy=0 0 0 -> xyz=-0.088054 -0.032677 -0.040824 rpy=0 0 0
- joint Rigid2: origin xyz=-0.121419 -0.029614 -0.228023 rpy=0 0 0 -> xyz=-0.088054 -0.032677 -0.258325 rpy=0 0 0
- joint arm1: origin xyz=0.313459 0.047886 -0.119273 rpy=0 0 0 -> xyz=0.346824 0.044823 -0.149575 rpy=0 0 0
- joint arm2: origin xyz=-0.014432 0.088193 -0.006 rpy=0 0 0 -> xyz=-0.014431 0.088193 -0.006 rpy=0 0 0
- joint arm3: origin xyz=-0.398022 0.039823 0.0 rpy=0 0 0 -> xyz=-0.398023 0.039823 0.0 rpy=0 0 0
