Commit message: Updated model to have T265 and D435i approximate models - T265 is just a stereo camera, without fisheye lenses though.

File: exp_description/model/simple.urdf (robot description, URDF)
Before this commit: robot simple, 5 links, 4 joints
Links:
- removed link camera
- added link D435i, mass 0.05; collision box size=0.04 0.04 0.04; visual box size=0.04 0.04 0.04
- added link T265, mass 0.05; collision box size=0.04 0.06 0.04; visual box size=0.04 0.06 0.04
Joints:
- removed joint camera
- added joint D435i: type fixed, parent body, child D435i, origin xyz=0.16 0 0.09
- added joint T265: type fixed, parent body, child T265, origin xyz=0.16 0 0.05

Commit message: Tried using differential track odometry instead of visual odometry

File: exp_description/model/simple.urdf (robot description, URDF)
Before this commit: robot simple, 6 links, 5 joints
Links:
- removed link D435i
- removed link T265
- added link D435i_link, mass 0.05; collision box size=0.04 0.04 0.04; visual box size=0.04 0.04 0.04
- added link T265_link, mass 0.05; collision box size=0.04 0.06 0.04; visual box size=0.04 0.06 0.04
- link body: mass 0.5 -> 1; geometry collision box size=0.6 0.3 0.2; collision sphere radius=0.1
- link wheel_left: mass 0.1 -> 0.5; geometry collision cylinder length=0.05 radius=0.15; visual cylinder length=0.05 radius=0.15
- link wheel_right: mass 0.1 -> 0.5; geometry collision cylinder length=0.05 radius=0.15; visual cylinder length=0.05 radius=0.15
Joints:
- removed joint D435i
- removed joint T265
- added joint D435i_joint: type fixed, parent body, child D435i_link, origin xyz=0.08 0 0.19
- added joint T265_joint: type fixed, parent body, child T265_link, origin xyz=0.08 0 0.15
- joint wheel_left: origin xyz=0 0.2 0 rpy=-1.571 0 0 -> xyz=0 0.15 0 rpy=-1.571 0 0
- joint wheel_right: origin xyz=0 -0.2 0 rpy=1.571 0 0 -> xyz=0 -0.15 0 rpy=1.571 0 0
