Commit message: Copied new urdf and meshes. Tidied up urdf.

File: arbie_description/model/arbie_original.urdf (robot description, URDF)
Before this commit: robot arbie, 28 links, 27 joints
Links:
- removed link arm_base_link
- removed link arm_lower_link
- removed link arm_upper_link
- removed link body_link
- removed link camera_d435_link
- removed link camera_mount_leg_1_link
- removed link camera_mount_leg_2_link
- removed link camera_mount_link
- removed link camera_t265_link
- removed link flipper_front_left_link
- removed link flipper_front_right_link
- removed link flipper_rear_left_link
- removed link flipper_rear_right_link
- removed link gripper_base_link
- removed link gripper_left_contact_link
- removed link gripper_left_driver_link
- removed link gripper_left_linkage_link
- removed link gripper_right_contact_link
- removed link gripper_right_driver_link
- removed link gripper_right_linkage_link
- removed link tracks_left_link
- removed link tracks_left_wheel_link
- removed link tracks_right_link
- removed link tracks_right_wheel_link
- removed link wrist_base_link
- removed link wrist_pitch_link
- removed link wrist_yaw_link
- added link Arm_link_1_1, mass 9.290217371436244; collision mesh filename=package://arbie_description/meshes/Arm_link_1_1_m-binary.stl; visual mesh filename=package://arbie_description/meshes/Arm_link_1_1_m-binary.stl
- added link Arm_link_2_1, mass 3.0631873001334227; collision mesh filename=package://arbie_description/meshes/Arm_link_2_1_m-binary.stl; visual mesh filename=package://arbie_description/meshes/Arm_link_2_1_m-binary.stl
- added link Arm_rotation_1, mass 3.3465093478653403; collision mesh filename=package://arbie_description/meshes/Arm_rotation_1_m-binary.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; visual mesh filename=package://arbie_description/meshes/Arm_rotation_1_m-binary.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
- added link Cam_mount_1, mass 0.10512980225278633; collision mesh filename=package://arbie_description/meshes/Cam_mount_1_m-binary.stl; visual mesh filename=package://arbie_description/meshes/Cam_mount_1_m-binary.stl
- added link D435_1, mass 0.3380578483539848; collision mesh filename=package://arbie_description/meshes/D435_1_m-binary.stl; visual mesh filename=package://arbie_description/meshes/D435_1_m-binary.stl
- added link Flipper_FL_1, mass 13.868020437393678; collision mesh filename=package://arbie_description/meshes/Flipper_FL_1_m-binary.stl; visual mesh filename=package://arbie_description/meshes/Flipper_FL_1_m-binary.stl
- added link Flipper_FR_1, mass 13.868020437393694; collision mesh filename=package://arbie_description/meshes/Flipper_FR_1_m-binary.stl; visual mesh filename=package://arbie_description/meshes/Flipper_FR_1_m-binary.stl
- added link Flipper_RL_1, mass 13.868020437393671; collision mesh filename=package://arbie_description/meshes/Flipper_RL_1_m-binary.stl; visual mesh filename=package://arbie_description/meshes/Flipper_RL_1_m-binary.stl
- added link Flipper_RR_1, mass 13.868020437393698; collision mesh filename=package://arbie_description/meshes/Flipper_RR_1_m-binary.stl; visual mesh filename=package://arbie_description/meshes/Flipper_RR_1_m-binary.stl
- added link Leg_1_1, mass 0.011972469965960587; collision mesh filename=package://arbie_description/meshes/Leg_1_1_m-binary.stl; visual mesh filename=package://arbie_description/meshes/Leg_1_1_m-binary.stl
- added link Leg_2_1, mass 0.011972469965960601; collision mesh filename=package://arbie_description/meshes/Leg_2_1_m-binary.stl; visual mesh filename=package://arbie_description/meshes/Leg_2_1_m-binary.stl
- added link T265_1, mass 0.11087104010777465; collision mesh filename=package://arbie_description/meshes/T265_1_m-binary.stl; visual mesh filename=package://arbie_description/meshes/T265_1_m-binary.stl
- added link Tracks_L_1, mass 44.76242127990538; collision mesh filename=package://arbie_description/meshes/Tracks_L_1_m-binary.stl; visual mesh filename=package://arbie_description/meshes/Tracks_L_1_m-binary.stl
- added link Tracks_R_1, mass 44.76242127990538; collision mesh filename=package://arbie_description/meshes/Tracks_R_1_m-binary.stl; visual mesh filename=package://arbie_description/meshes/Tracks_R_1_m-binary.stl
- added link equivalent_wheel_L_1, mass 1.3872095061007428; collision mesh filename=package://arbie_description/meshes/equivalent_wheel_L_1_m-b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; visual mesh filename=package://arbie_description/meshes/equivalent_wheel_L_1_m-b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
- added link equivalent_wheel_R_1, mass 1.3872095061007428; collision mesh filename=package://arbie_description/meshes/equivalent_wheel_R_1_m-b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; visual mesh filename=package://arbie_description/meshes/equivalent_wheel_R_1_m-b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
- added link gripper_mount_1, mass 0.6706735500880907; collision mesh filename=package://arbie_description/meshes/gripper_mount_1_m-binary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; visual mesh filename=package://arbie_description/meshes/gripper_mount_1_m-binary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
- added link l_finger_1, mass 0.023712538812289255; collision mesh filename=package://arbie_description/meshes/l_finger_1_m-binary.stl; visual mesh filename=package://arbie_description/meshes/l_finger_1_m-binary.stl
- added link l_link1_1, mass 0.013747989643093032; collision mesh filename=package://arbie_description/meshes/l_link1_1_m-binary.stl; visual mesh filename=package://arbie_description/meshes/l_link1_1_m-binary.stl
- added link l_link2_1, mass 0.00386409068463368; collision mesh filename=package://arbie_description/meshes/l_link2_1_m-binary.stl; visual mesh filename=package://arbie_description/meshes/l_link2_1_m-binary.stl
- added link pitch_mount_1, mass 0.08039663104912372; collision mesh filename=package://arbie_description/meshes/pitch_mount_1_m-binary.s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; visual mesh filename=package://arbie_description/meshes/pitch_mount_1_m-binary.s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
- added link r_finger_1, mass 0.023712538812289255; collision mesh filename=package://arbie_description/meshes/r_finger_1_m-binary.stl; visual mesh filename=package://arbie_description/meshes/r_finger_1_m-binary.stl
- added link r_link1_1, mass 0.01374798583124482; collision mesh filename=package://arbie_description/meshes/r_link1_1_m-binary.stl; visual mesh filename=package://arbie_description/meshes/r_link1_1_m-binary.stl
- added link roll_yaw_servo_1, mass 0.6469480906726006; collision mesh filename=package://arbie_description/meshes/roll_yaw_servo_1_m-binar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; visual mesh filename=package://arbie_description/meshes/roll_yaw_servo_1_m-binar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
- added link wrist_base_1, mass 0.9490572232520995; collision mesh filename=package://arbie_description/meshes/wrist_base_1_m-binary.stl; visual mesh filename=package://arbie_description/meshes/wrist_base_1_m-binary.stl
- link base_link: mass None -> 132.38352048208554; geometry collision mesh filename=package://arbie_description/meshes/base_link_m-binary.stl; visual mesh filename=package://arbie_description/meshes/base_link_m-binary.stl
Joints:
- removed joint arm_1_joint
- removed joint arm_2_joint
- removed joint arm_3_joint
- removed joint base_joint
- removed joint camera_mount_joint
- removed joint flipper_front_left_joint
- removed joint flipper_front_right_joint
- removed joint flipper_rear_left_joint
- removed joint flipper_rear_right_joint
- removed joint gripper_left_contact_dependent_joint
- removed joint gripper_left_driver_joint
- removed joint gripper_left_linkage_dependent_joint
- removed joint gripper_right_contact_dependent_joint
- removed joint gripper_right_driver_joint
- removed joint gripper_right_linkage_dependent_joint
- removed joint rigid_arm_upper_to_wrist_base_joint
- removed joint rigid_body_to_camera_mount_leg_1_joint
- removed joint rigid_body_to_camera_mount_leg_2_joint
- removed joint rigid_body_to_tracks_left_joint
- removed joint rigid_body_to_tracks_right_joint
- removed joint rigid_camera_mount_to_camera_d435_joint
- removed joint rigid_camera_mount_to_camera_t265_joint
- removed joint tracks_left_joint
- removed joint tracks_right_joint
- removed joint wrist_pitch_joint
- removed joint wrist_roll_joint
- removed joint wrist_yaw_joint
- added joint Rev28: type continuous, parent Leg_1_1, child Cam_mount_1, origin xyz=-0.004 0.02575 0.0 rpy=0 0 0, axis 0.01 0.0 -0.0
- added joint Rev31: type continuous, parent Tracks_R_1, child Flipper_FR_1, origin xyz=-0.05 0.005403 0.23 rpy=0 0 0, axis 0.01 -0.0 0.0
- added joint Rev32: type continuous, parent Tracks_R_1, child Flipper_RR_1, origin xyz=-0.05 0.005403 -0.23 rpy=0 0 0, axis 0.01 -0.0 0.0
- added joint Rev33: type continuous, parent Tracks_L_1, child Flipper_FL_1, origin xyz=0.05 0.005403 0.23 rpy=0 0 0, axis 0.01 0.0 -0.0
- added joint Rev34: type continuous, parent Tracks_L_1, child Flipper_RL_1, origin xyz=0.05 0.005403 -0.23 rpy=0 0 0, axis 0.01 0.0 -0.0
- added joint Rev35: type continuous, parent base_link, child Arm_rotation_1, origin xyz=-0.000694 0.107101 0.186272 rpy=0 0 0, axis -0.0 -0.01 0.0
- added joint Rev36: type continuous, parent Arm_rotation_1, child Arm_link_1_1, origin xyz=0.0535 0.067 0.000223 rpy=0 0 0, axis 0.01 0.0 -0.0
- added joint Rev37: type continuous, parent Arm_link_1_1, child Arm_link_2_1, origin xyz=-0.033 0.035 -0.45 rpy=0 0 0, axis -0.01 -0.0 0.0
- added joint Rev39: type continuous, parent wrist_base_1, child pitch_mount_1, origin xyz=0.0334 0.0 0.0535 rpy=0 0 0, axis -0.01 -0.0 -0.0
- added joint Rev40: type continuous, parent pitch_mount_1, child roll_yaw_servo_1, origin xyz=-0.0333 -0.01845 0.063124 rpy=0 0 0, axis 0.0 -0.01 -0.0
- added joint Rev41: type continuous, parent roll_yaw_servo_1, child gripper_mount_1, origin xyz=0.0 0.019 0.0454 rpy=0 0 0, axis -0.0 -0.0 0.01
- added joint Rev42: type continuous, parent gripper_mount_1, child r_link1_1, origin xyz=0.016 0.019 0.0487 rpy=0 0 0, axis -0.0 0.01 0.0
- added joint Rev43: type continuous, parent gripper_mount_1, child l_link1_1, origin xyz=-0.016 0.019 0.0487 rpy=0 0 0, axis -0.0 0.01 0.0
- added joint Rev44: type continuous, parent l_link1_1, child l_finger_1, origin xyz=0.0 -0.0024 0.035 rpy=0 0 0, axis 0.0 -0.01 -0.0
- added joint Rev45: type continuous, parent r_link1_1, child r_finger_1, origin xyz=0.0 -0.0024 0.035 rpy=0 0 0, axis -0.0 0.01 0.0
- added joint Rev46: type continuous, parent gripper_mount_1, child l_link2_1, origin xyz=-0.039616 -0.006 0.0302 rpy=0 0 0, axis 0.0 -0.01 -0.0
- added joint Rigid22: type fixed, parent base_link, child Tracks_L_1, origin xyz=0.123306 0.019326 -0.010978 rpy=0 0 0
- added joint Rigid23: type fixed, parent base_link, child Tracks_R_1, origin xyz=-0.124694 0.019326 -0.010978 rpy=0 0 0
- added joint Rigid24: type fixed, parent Tracks_R_1, child equivalent_wheel_R_1, origin xyz=-0.02 0.0 0.0 rpy=0 0 0
- added joint Rigid25: type fixed, parent Tracks_L_1, child equivalent_wheel_L_1, origin xyz=0.02 0.0 0.0 rpy=0 0 0
- added joint Rigid26: type fixed, parent base_link, child Leg_1_1, origin xyz=0.037807 0.048101 0.262572 rpy=0 0 0
- added joint Rigid27: type fixed, parent base_link, child Leg_2_1, origin xyz=-0.039194 0.048101 0.262572 rpy=0 0 0
- added joint Rigid29: type fixed, parent Cam_mount_1, child D435_1, origin xyz=-0.012557 -0.073851 -0.287572 rpy=0 0 0
- added joint Rigid30: type fixed, parent Cam_mount_1, child T265_1, origin xyz=-0.01763 -0.0135 0.014 rpy=0 0 0
- added joint Rigid38: type fixed, parent Arm_link_2_1, child wrist_base_1, origin xyz=-0.017 0.035 0.225 rpy=0 0 0
