Commit message: Some launch file changes. Re-generated moveit config

File: arbie_description/model/arbie.urdf (robot description, URDF)
Before this commit: robot rescue, 16 links, 15 joints
Links:
- link arm_base_1: geometry collision mesh filename=package://arbie_description/meshes/arm_base_1_m-binary.stl; visual mesh filename=package://arbie_description/meshes/arm_base_1_m-binary.stl
- link arm_lower_1: geometry collision mesh filename=package://arbie_description/meshes/arm_lower_1_m-binary.stl; visual mesh filename=package://arbie_description/meshes/arm_lower_1_m-binary.stl
- link arm_upper_1: geometry collision mesh filename=package://arbie_description/meshes/arm_upper_1_m-binary.stl; visual mesh filename=package://arbie_description/meshes/arm_upper_1_m-binary.stl
- link flipper_front_left_1: geometry collision cylinder length=0.05 radius=0.24; visual mesh filename=package://arbie_description/meshes/flipper_front_left_1_m-b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
- link flipper_front_right_1: geometry collision cylinder length=0.05 radius=0.24; visual mesh filename=package://arbie_description/meshes/flipper_front_right_1_m-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
- link flipper_rear_left_1: geometry collision cylinder length=0.05 radius=0.24; visual mesh filename=package://arbie_description/meshes/flipper_rear_left_1_m-bi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
- link flipper_rear_right_1: geometry collision cylinder length=0.05 radius=0.24; visual mesh filename=package://arbie_description/meshes/flipper_rear_right_1_m-b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
- link gripper_1: geometry collision mesh filename=package://arbie_description/meshes/gripper_1_m-binary.stl; visual mesh filename=package://arbie_description/meshes/gripper_1_m-binary.stl
- link left_belt_1: geometry collision mesh filename=package://arbie_description/meshes/left_belt_1_m-binary.stl; visual mesh filename=package://arbie_description/meshes/left_belt_1_m-binary.stl
- link main_body: geometry collision mesh filename=package://arbie_description/meshes/base_link_m-binary.stl; visual mesh filename=package://arbie_description/meshes/base_link_m-binary.stl
- link right_belt_1: geometry collision mesh filename=package://arbie_description/meshes/right_belt_1_m-binary.stl; visual mesh filename=package://arbie_description/meshes/right_belt_1_m-binary.stl
- link wrist_pitch_1: geometry collision mesh filename=package://arbie_description/meshes/wrist_pitch_1_m-binary.s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; visual mesh filename=package://arbie_description/meshes/wrist_pitch_1_m-binary.s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
- link wrist_yaw_1: geometry collision mesh filename=package://arbie_description/meshes/wrist_yaw_1_m-binary.stl; visual mesh filename=package://arbie_description/meshes/wrist_yaw_1_m-binary.stl

Commit message: Regenerated moveit config, made various tweaks

File: arbie_description/model/arbie.urdf (robot description, URDF)
Before this commit: robot rescue, 16 links, 15 joints
Links:
- link flipper_front_left_1: geometry collision mesh filename=package://arbie_description/meshes/flipper_front_left_1_m-b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; visual mesh filename=package://arbie_description/meshes/flipper_front_left_1_m-b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
- link flipper_front_right_1: geometry collision mesh filename=package://arbie_description/meshes/flipper_front_right_1_m-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; visual mesh filename=package://arbie_description/meshes/flipper_front_right_1_m-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
- link flipper_rear_left_1: geometry collision mesh filename=package://arbie_description/meshes/flipper_rear_left_1_m-bi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; visual mesh filename=package://arbie_description/meshes/flipper_rear_left_1_m-bi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
- link flipper_rear_right_1: geometry collision mesh filename=package://arbie_description/meshes/flipper_rear_right_1_m-b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; visual mesh filename=package://arbie_description/meshes/flipper_rear_right_1_m-b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

Commit message: Renamed meshes

File: arbie_description/model/arbie.urdf (robot description, URDF)
Before this commit: robot arbie, 28 links, 27 joints
Links:
- link arm_base_link: geometry collision mesh filename=package://arbie_description/meshes/arm_base.stl; visual mesh filename=package://arbie_description/meshes/arm_base.stl
- link arm_lower_link: geometry collision mesh filename=package://arbie_description/meshes/arm_lower.stl; visual mesh filename=package://arbie_description/meshes/arm_lower.stl
- link arm_upper_link: geometry collision mesh filename=package://arbie_description/meshes/arm_upper.stl; visual mesh filename=package://arbie_description/meshes/arm_upper.stl
- link body_link: geometry collision mesh filename=package://arbie_description/meshes/body.stl; visual mesh filename=package://arbie_description/meshes/body.stl
- link camera_d435_link: geometry collision mesh filename=package://arbie_description/meshes/camera_d435.stl; visual mesh filename=package://arbie_description/meshes/camera_d435.stl
- link camera_mount_leg_1_link: geometry collision mesh filename=package://arbie_description/meshes/camera_mount_leg_1.stl; visual mesh filename=package://arbie_description/meshes/camera_mount_leg_1.stl
- link camera_mount_leg_2_link: geometry collision mesh filename=package://arbie_description/meshes/camera_mount_leg_2.stl; visual mesh filename=package://arbie_description/meshes/camera_mount_leg_2.stl
- link camera_mount_link: geometry collision mesh filename=package://arbie_description/meshes/camera_mount.stl; visual mesh filename=package://arbie_description/meshes/camera_mount.stl
- link camera_t265_link: geometry collision mesh filename=package://arbie_description/meshes/camera_t265.stl; visual mesh filename=package://arbie_description/meshes/camera_t265.stl
- link flipper_front_left_link: geometry collision mesh filename=package://arbie_description/meshes/flipper_front_left.stl; visual mesh filename=package://arbie_description/meshes/flipper_front_left.stl
- link flipper_front_right_link: geometry collision mesh filename=package://arbie_description/meshes/flipper_front_right.stl; visual mesh filename=package://arbie_description/meshes/flipper_front_right.stl
- link flipper_rear_left_link: geometry collision mesh filename=package://arbie_description/meshes/flipper_rear_left.stl; visual mesh filename=package://arbie_description/meshes/flipper_rear_left.stl
- link flipper_rear_right_link: geometry collision mesh filename=package://arbie_description/meshes/flipper_rear_right.stl; visual mesh filename=package://arbie_description/meshes/flipper_rear_right.stl
- link gripper_base_link: geometry collision mesh filename=package://arbie_description/meshes/gripper_base.stl; visual mesh filename=package://arbie_description/meshes/gripper_base.stl
- link gripper_left_contact_link: geometry collision mesh filename=package://arbie_description/meshes/gripper_left_contact.stl; visual mesh filename=package://arbie_description/meshes/gripper_left_conctact.stl
- link gripper_left_driver_link: geometry collision mesh filename=package://arbie_description/meshes/gripper_left_driver.stl; visual mesh filename=package://arbie_description/meshes/gripper_left_driver.stl
- link gripper_left_linkage_link: geometry collision mesh filename=package://arbie_description/meshes/gripper_left_linkage.stl; visual mesh filename=package://arbie_description/meshes/gripper_left_linkage.stl
- link gripper_right_contact_link: geometry collision mesh filename=package://arbie_description/meshes/gripper_right_contact.stl; visual mesh filename=package://arbie_description/meshes/gripper_right_contact.stl
- link gripper_right_driver_link: geometry collision mesh filename=package://arbie_description/meshes/gripper_right_driver.stl; visual mesh filename=package://arbie_description/meshes/gripper_right_driver.stl
- link gripper_right_linkage_link: geometry collision mesh filename=package://arbie_description/meshes/gripper_right_linkage.stl; visual mesh filename=package://arbie_description/meshes/gripper_right_linkage.stl
- link tracks_left_link: geometry collision mesh filename=package://arbie_description/meshes/tracks_left.stl; visual mesh filename=package://arbie_description/meshes/tracks_left.stl
- link tracks_left_wheel_link: geometry collision mesh filename=package://arbie_description/meshes/tracks_left_wheel.stl; visual mesh filename=package://arbie_description/meshes/tracks_left_wheel.stl
- link tracks_right_link: geometry collision mesh filename=package://arbie_description/meshes/tracks_right.stl; visual mesh filename=package://arbie_description/meshes/tracks_right.stl
- link tracks_right_wheel_link: geometry collision mesh filename=package://arbie_description/meshes/tracks_right_wheel.stl; visual mesh filename=package://arbie_description/meshes/tracks_right_wheel.stl
- link wrist_base_link: geometry collision mesh filename=package://arbie_description/meshes/wrist_base.stl; visual mesh filename=package://arbie_description/meshes/wrist_base.stl
- link wrist_pitch_link: geometry collision mesh filename=package://arbie_description/meshes/wrist_pitch.stl; visual mesh filename=package://arbie_description/meshes/wrist_pitch.stl
- link wrist_yaw_link: geometry collision mesh filename=package://arbie_description/meshes/wrist_yaw.stl; visual mesh filename=package://arbie_description/meshes/wrist_yaw.stl

Commit message: Added mimic tag to dependent joints

File: arbie_description/model/arbie.urdf (robot description, URDF)
Before this commit: robot arbie, 28 links, 27 joints
Joints:
- joint gripper_left_contact_dependent_joint: mimic (none) -> joint=gripper_left_driver_joint
- joint gripper_left_linkage_dependent_joint: mimic (none) -> joint=gripper_left_driver_joint
- joint gripper_right_contact_dependent_joint: mimic (none) -> joint=gripper_right_driver_joint
- joint gripper_right_linkage_dependent_joint: mimic (none) -> joint=gripper_right_driver_joint

Commit message: Urdf model working

File: arbie_description/model/arbie.urdf (robot description, URDF)
Before this commit: robot arbie, 28 links, 27 joints
Links:
- link gripper_left_contact_link: geometry collision mesh filename=package://arbie_description/meshes/gripper_left_contact.stl; visual mesh filename=package://arbie_description/meshes/gripper_left_contact.stl
Joints:
- joint base_joint: origin xyz=0 0 0.5 rpy=0 1.57 0 -> xyz=0.01 0 0.075 rpy=1.5708 0 1.5708
- joint gripper_left_contact_dependent_joint: axis 0 -1 0 -> 0 1 0; mimic joint=gripper_left_driver_joint -> joint=gripper_left_driver_joint multiplier=-1
- joint gripper_left_linkage_dependent_joint: axis 0 -1 0 -> 0 1 0; mimic joint=gripper_left_driver_joint -> joint=gripper_left_driver_joint multiplier=1
- joint gripper_right_contact_dependent_joint: mimic joint=gripper_right_driver_joint -> joint=gripper_right_driver_joint multiplier=-1
- joint gripper_right_linkage_dependent_joint: axis 0 -1 0 -> 0 1 0; mimic joint=gripper_right_driver_joint -> joint=gripper_right_driver_joint multiplier=1

Commit message: Started testing out arm control

File: arbie_description/model/arbie.urdf (robot description, URDF)
Before this commit: robot arbie, 28 links, 27 joints
Joints:
- removed joint gripper_left_driver_joint
- removed joint gripper_right_driver_joint
- added joint gripper_joint: type continuous, parent gripper_base_link, child gripper_right_driver_link, origin xyz=0.016 0.019 0.0487 rpy=0 0 0, axis 0 1 0
- added joint gripper_mimic_joint: type continuous, parent gripper_base_link, child gripper_left_driver_link, origin xyz=-0.016 0.019 0.0487 rpy=0 0 0, axis 0 1 0, mimic joint=gripper_joint multiplier=-1
- joint gripper_left_contact_dependent_joint: mimic joint=gripper_left_driver_joint multiplier=-1 -> joint=gripper_joint multiplier=1
- joint gripper_left_linkage_dependent_joint: mimic joint=gripper_left_driver_joint multiplier=1 -> joint=gripper_joint multiplier=-1
- joint gripper_right_contact_dependent_joint: mimic joint=gripper_right_driver_joint multiplier=-1 -> joint=gripper_joint multiplier=-1
- joint gripper_right_linkage_dependent_joint: mimic joint=gripper_right_driver_joint multiplier=1 -> joint=gripper_joint multiplier=1

Commit message: Calibrated gripper joints

File: arbie_description/model/arbie.urdf (robot description, URDF)
Before this commit: robot arbie, 28 links, 27 joints
Joints:
- joint gripper_joint: origin xyz=0.016 0.019 0.0487 rpy=0 0 0 -> xyz=0.016 0.019 0.0487 rpy=0 -0.348 0
- joint gripper_left_contact_dependent_joint: origin xyz=0.0 -0.0024 0.035 rpy=0 0 0 -> xyz=0.0 -0.0024 0.035 rpy=0 -0.348 0
- joint gripper_left_linkage_dependent_joint: origin xyz=-0.039616 -0.006 0.0302 rpy=0 0 0 -> xyz=-0.039616 -0.006 0.0302 rpy=0 0.348 0
- joint gripper_mimic_joint: origin xyz=-0.016 0.019 0.0487 rpy=0 0 0 -> xyz=-0.016 0.019 0.0487 rpy=0 0.348 0
- joint gripper_right_contact_dependent_joint: origin xyz=0.0 -0.0024 0.035 rpy=0 0 0 -> xyz=0.0 -0.0024 0.035 rpy=0 0.348 0
- joint gripper_right_linkage_dependent_joint: origin xyz=0.039616 -0.006 0.0302 rpy=0 0 0 -> xyz=0.039616 -0.006 0.0302 rpy=0 -0.348 0

Commit message: Added arm calibration.

File: arbie_description/model/arbie.urdf (robot description, URDF)
Before this commit: robot arbie, 28 links, 27 joints
Joints:
- joint arm_2_joint: axis 1 0 0 -> -1 0 0
- joint arm_3_joint: axis -1 0 0 -> 1 0 0
- joint wrist_pitch_joint: axis -1 0 0 -> 1 0 0
- joint wrist_roll_joint: origin xyz=0.0 0.019 0.0454 rpy=0 0 0 -> xyz=0.0 0.019 0.0454 rpy=0 0 -1.5708

Commit message: Calibrated arm motors with gear ratios

File: arbie_description/model/arbie.urdf (robot description, URDF)
Before this commit: robot arbie, 28 links, 27 joints
Joints:
- joint arm_2_joint: axis -1 0 0 -> 1 0 0
- joint arm_3_joint: axis 1 0 0 -> -1 0 0

Commit message: Fixed joint between upper arm wrist base, and arm_1_joint axis.

File: arbie_description/model/arbie.urdf (robot description, URDF)
Before this commit: robot arbie, 28 links, 27 joints
Joints:
- joint arm_1_joint: axis 0 -1 0 -> 0 1 0
- joint rigid_arm_upper_to_wrist_base_joint: origin xyz=-0.017 0.035 0.225 rpy=0 0 0 -> xyz=-0.017 0.035 0.27 rpy=0 0 0

Commit message: Started adding position controllers. Tweaking ros model.

File: arbie_description/model/arbie.urdf (robot description, URDF)
Before this commit: robot arbie, 28 links, 27 joints
Joints:
- removed joint flipper_front_left_joint
- removed joint flipper_front_right_joint
- removed joint flipper_rear_left_joint
- removed joint flipper_rear_right_joint
- added joint flipper_front_joint: type continuous, parent tracks_right_link, child flipper_front_right_link, origin xyz=-0.05 0.005403 0.23 rpy=0 0 0, axis 1 0 0
- added joint flipper_front_mimic_joint: type continuous, parent tracks_left_link, child flipper_front_left_link, origin xyz=0.05 0.005403 0.23 rpy=0 0 0, axis 1 0 0, mimic joint=flipper_front_joint
- added joint flipper_rear_joint: type continuous, parent tracks_right_link, child flipper_rear_right_link, origin xyz=-0.05 0.005403 -0.23 rpy=0 0 0, axis 1 0 0
- added joint flipper_rear_mimic_joint: type continuous, parent tracks_left_link, child flipper_rear_left_link, origin xyz=0.05 0.005403 -0.23 rpy=0 0 0, axis 1 0 0, mimic joint=flipper_rear_joint

Commit message: Changed urdf to have fixed joint between left and right flippers

File: arbie_description/model/arbie.urdf (robot description, URDF)
Before this commit: robot arbie, 28 links, 27 joints
Joints:
- removed joint flipper_front_mimic_joint
- removed joint flipper_rear_mimic_joint
- added joint rigid_flipper_front_right_to_flipper_front_left: type fixed, parent flipper_front_right_link, child flipper_front_left_link, origin xyz=0.347996 0 0 rpy=0 0 0
- added joint rigid_flipper_rear_right_to_flipper_rear_left: type fixed, parent flipper_rear_right_link, child flipper_rear_left_link, origin xyz=0.347996 0 0 rpy=0 0 0
