Commit message: arbie_base works in simulation

File: arbie_description/model/arbie_base_sim.urdf.xacro (robot description, xacro)
@@ -8,4 +8,6 @@
 <!-- Differential drive wheels and caster. Approximates track kinematics -->
 <xacro:include filename='components/tracks_sim.urdf'/>
+<gazebo>
 <plugin name="gazebo_ros_control" filename="libgazebo_ros_control.so"/>
+</gazebo>
 </robot>

File: arbie_description/model/components/base.urdf.xacro (robot description, xacro)
@@ -205,5 +205,5 @@
 </joint>
 <!-- CAMERA MOUNT JOINT -->
-<joint name="camera_mount_joint" type="continuous">
+<joint name="camera_tilt_joint" type="continuous">
   <origin rpy="0 0 0" xyz="-0.004 0.02575 0.0"/>
   <parent link="camera_mount_leg_1_link"/>
@@ -213,9 +213,9 @@
 <transmission name="camera_mount_transmission">
   <type>transmission_interface/SimpleTransmission</type>
-  <joint name="camera_mount_joint">
-    <hardwareInterface>hardware_interface/${pos_interface}</hardwareInterface>
+  <joint name="camera_tilt_joint">
+    <hardwareInterface>hardware_interface/PositionJointInterface</hardwareInterface>
   </joint>
   <actuator name="camera_mount_actuator">
-    <hardwareInterface>${pos_interface}</hardwareInterface>
+    <hardwareInterface>PositionJointInterface</hardwareInterface>
     <mechanicalReduction>1</mechanicalReduction>
   </actuator>

File: arbie_description/model/components/wheel.urdf.xacro (robot description, xacro)
@@ -11,5 +11,5 @@
 </visual>
 <collision>
-    <origin xyz="0 0 0" rpy="0 0 ${pi/2}"/>
+    <origin xyz="0 0 0" rpy="0 ${pi/2} 0"/>
     <geometry>
         <cylinder length="${length}" radius="${radius}"/>
