Commit message: Tweaking controllers for simulation

File: arbie_description/model/arbie_sim.urdf.xacro (robot description, xacro)
@@ -4,5 +4,5 @@
 <!-- Flippers -->
 <xacro:include filename='components/flippers.urdf.xacro'/>
-<xacro:flippers pos_interface='PositionJointInterface' vel_interface='VelocityJointInterface'/>
+<xacro:flippers pos_interface='EffortJointInterface' vel_interface='EffortJointInterface'/>
 <!-- Arm, wrist, gripper -->
 <xacro:include filename='components/arm.urdf.xacro'/>

File: arbie_description/model/components/arm.urdf.xacro (robot description, xacro)
@@ -165,4 +165,5 @@
   </collision>
 </link>
+<!--
 <link name="gripper_right_linkage_link">
   <inertial>
@@ -173,5 +174,4 @@
   <visual>
     <origin rpy="0 0 0" xyz="0.015 -0.485 -0.09"/>
-    <!--<origin rpy="0 0 0" xyz="0.03671 -0.238651 -0.153719"/>-->
     <geometry>
       <mesh filename="package://arbie_description/meshes/gripper_right_linkage.stl"/>
@@ -206,4 +206,5 @@
   </collision>
 </link>
+-->
 <link name="gripper_left_driver_link">
   <inertial>
@@ -226,4 +227,5 @@
   </collision>
 </link>
+<!--
 <link name="gripper_left_contact_link">
   <inertial>
@@ -266,4 +268,5 @@
   </collision>
 </link>
+-->
 <!-- RIGID JOINTS -->
 <joint name="rigid_arm_upper_to_wrist_base_joint" type="fixed">
@@ -371,5 +374,5 @@
 </transmission>
 <!-- GRIPPER DRIVEN JOINTS -->
-<joint name="gripper_joint" type="continuous">
+<joint name="gripper_right_joint" type="continuous">
   <origin rpy="0 -0.348 0" xyz="0.016 0.019 0.0487"/>
   <parent link="gripper_base_link"/>
@@ -379,29 +382,25 @@
 <transmission name="gripper_right_driver_transmission">
   <type>transmission_interface/SimpleTransmission</type>
-  <joint name="gripper_joint">
-    <hardwareInterface>hardware_interface/${pos_interface}</hardwareInterface>
+  <joint name="gripper_right_joint">
+    <hardwareInterface>hardware_interface/EffortJointInterface</hardwareInterface>
   </joint>
   <actuator name="gripper_right_driver_actuator">
-    <hardwareInterface>${pos_interface}</hardwareInterface>
-    <mechanicalReduction>1</mechanicalReduction>
-  </actuator>
-</transmission>
-<!-- Also driven, but treat these two joints as the same
-Controller drives them together. Make this joint mimic
-the other -->
-<joint name="gripper_mimic_joint" type="continuous">
+    <hardwareInterface>EffortJointInterface</hardwareInterface>
+    <mechanicalReduction>1</mechanicalReduction>
+  </actuator>
+</transmission>
+<joint name="gripper_left_joint" type="continuous">
   <origin rpy="0 0.348 0" xyz="-0.016 0.019 0.0487"/>
   <parent link="gripper_base_link"/>
   <child link="gripper_left_driver_link"/>
   <axis xyz="0 1 0"/>
-  <mimic joint="gripper_joint" multiplier="-1"/>
 </joint>
 <transmission name="gripper_left_driver_transmission">
   <type>transmission_interface/SimpleTransmission</type>
-  <joint name="gripper_mimic_joint">
-    <hardwareInterface>hardware_interface/${pos_interface}</hardwareInterface>
+  <joint name="gripper_left_joint">
+    <hardwareInterface>hardware_interface/EffortJointInterface</hardwareInterface>
   </joint>
   <actuator name="gripper_left_driver_actuator">
-    <hardwareInterface>${pos_interface}</hardwareInterface>
+    <hardwareInterface>EffortJointInterface</hardwareInterface>
     <mechanicalReduction>1</mechanicalReduction>
   </actuator>

File: arbie_description/model/components/flippers.urdf.xacro (robot description, xacro)
@@ -95,5 +95,5 @@
 </joint>
 <!-- FLIPPER JOINTS -->
-<joint name="flipper_front_joint" type="continuous">
+<joint name="flippers_front_joint" type="continuous">
   <origin rpy="0 0 0" xyz="-0.05 0.005403 0.23"/>
   <parent link="tracks_right_link"/>
@@ -101,15 +101,15 @@
   <axis xyz="1 0 0"/>
 </joint>
-<transmission name="flipper_front_transmission">
+<transmission name="flippers_front_transmission">
   <type>transmission_interface/SimpleTransmission</type>
-  <joint name="flipper_front_joint">
+  <joint name="flippers_front_joint">
     <hardwareInterface>hardware_interface/${vel_interface}</hardwareInterface>
   </joint>
-  <actuator name="flipper_front_actuator">
+  <actuator name="flippers_front_actuator">
     <hardwareInterface>${vel_interface}</hardwareInterface>
     <mechanicalReduction>1</mechanicalReduction>
   </actuator>
 </transmission>
-<joint name="flipper_rear_joint" type="continuous">
+<joint name="flippers_rear_joint" type="continuous">
   <origin rpy="0 0 0" xyz="-0.05 0.005403 -0.23"/>
   <parent link="tracks_right_link"/>
@@ -117,10 +117,10 @@
   <axis xyz="1 0 0"/>
 </joint>
-<transmission name="flipper_rear_transmission">
+<transmission name="flippers_rear_transmission">
   <type>transmission_interface/SimpleTransmission</type>
-  <joint name="flipper_rear_joint">
+  <joint name="flippers_rear_joint">
     <hardwareInterface>hardware_interface/${vel_interface}</hardwareInterface>
   </joint>
-  <actuator name="flipper_rear_actuator">
+  <actuator name="flippers_rear_actuator">
     <hardwareInterface>${vel_interface}</hardwareInterface>
     <mechanicalReduction>1</mechanicalReduction>
