Commit message: Trying to get extra joints to work

File: arbie_description/model/components/arm.urdf.xacro (robot description, xacro)
@@ -165,5 +165,4 @@
   </collision>
 </link>
-<!--
 <link name="gripper_right_linkage_link">
   <inertial>
@@ -227,5 +226,4 @@
   </collision>
 </link>
-<!--
 <link name="gripper_left_contact_link">
   <inertial>
@@ -268,5 +266,4 @@
   </collision>
 </link>
--->
 <!-- RIGID JOINTS -->
 <joint name="rigid_arm_upper_to_wrist_base_joint" type="fixed">
@@ -407,5 +404,4 @@
 </transmission>
 <!-- GRIPPER DEPENDENT JOINTS -->
-<!--
 <joint name="gripper_right_contact_dependent_joint" type="continuous">
   <origin rpy="0 0.348 0" xyz="0.0 -0.0024 0.035"/>
@@ -413,5 +409,5 @@
   <child link="gripper_right_contact_link"/>
   <axis xyz="0 1 0"/>
-  <mimic joint="gripper_joint" multiplier="-1"/>
+  <mimic joint="gripper_right_joint" multiplier="-1"/>
 </joint>
 <joint name="gripper_left_contact_dependent_joint" type="continuous">
@@ -420,5 +416,5 @@
   <child link="gripper_left_contact_link"/>
   <axis xyz="0 1 0"/>
-  <mimic joint="gripper_joint" multiplier="1"/>
+  <mimic joint="gripper_left_joint" multiplier="-1"/>
 </joint>
 <joint name="gripper_right_linkage_dependent_joint" type="continuous">
@@ -427,5 +423,5 @@
   <child link="gripper_right_linkage_link"/>
   <axis xyz="0 1 0"/>
-  <mimic joint="gripper_joint" multiplier="1"/>
+  <mimic joint="gripper_right_joint"/>
 </joint>
 <joint name="gripper_left_linkage_dependent_joint" type="continuous">
@@ -434,7 +430,21 @@
   <child link="gripper_left_linkage_link"/>
   <axis xyz="0 1 0"/>
-  <mimic joint="gripper_joint" multiplier="-1"/>
-</joint>
--->
+  <mimic joint="gripper_left_joint"/>
+</joint>
+<!-- GAZEBO ONLY JOINTS - CLOSE LOOP -->
+<gazebo>
+<joint name="gripper_right_linkage_dependent_2_joint" type="revolute">
+  <pose>0 0 0 0 0 0</pose>
+  <parent>gripper_right_linkage_link</parent>
+  <child>gripper_right_contact_link"</child>
+  <axis><xyz>0 1 0</xyz></axis>
+</joint>
+<joint name="gripper_left_linkage_dependent_2_joint" type="revolute">
+  <pose>0 0 0 0 0 0</pose>
+  <parent>gripper_left_linkage_link</parent>
+  <child>gripper_left_contact_link"</child>
+  <axis><xyz>0 1 0</xyz></axis>
+</joint>
+</gazebo>
 </xacro:macro>
 </to_include>

Commit message: Gripper extra joint work, but doesn't simulate well.

File: arbie_description/model/components/arm.urdf.xacro (robot description, xacro)
@@ -434,15 +434,37 @@
 <!-- GAZEBO ONLY JOINTS - CLOSE LOOP -->
 <gazebo>
-<joint name="gripper_right_linkage_dependent_2_joint" type="revolute">
+<joint name='gripper_left_linkage_dependent_joint2' type='revolute'>
+  <pose>-0.0235 -0.0225 -0.0185 0 0 0</pose>
+  <child>gripper_left_contact_link</child>
+  <parent>gripper_left_linkage_link</parent>
+  <axis>
+    <xyz>-4e-06 1 -4e-06</xyz>
+    <limit>
+      <lower>-1e+16</lower>
+      <upper>1e+16</upper>
+    </limit>
+    <dynamics>
+      <spring_reference>0</spring_reference>
+      <spring_stiffness>0</spring_stiffness>
+    </dynamics>
+    <use_parent_model_frame>1</use_parent_model_frame>
+  </axis>
+</joint>
+<joint name='gripper_right_linkage_dependent_joint2' type='revolute'>
   <pose>0.0235 -0.0225 -0.0185 0 0 0</pose>
+  <child>gripper_right_contact_link</child>
   <parent>gripper_right_linkage_link</parent>
-  <child>gripper_right_contact_link"</child>
-  <axis><xyz>0 1 0</xyz></axis>
-</joint>
-<joint name="gripper_left_linkage_dependent_2_joint" type="revolute">
-  <pose>0.0235 -0.0225 -0.0185 0 0 0</pose>
-  <parent>gripper_left_linkage_link</parent>
-  <child>gripper_left_contact_link"</child>
-  <axis><xyz>0 1 0</xyz></axis>
+  <axis>
+    <xyz>-4e-06 1 -4e-06</xyz>
+    <limit>
+      <lower>-1e+16</lower>
+      <upper>1e+16</upper>
+    </limit>
+    <dynamics>
+      <spring_reference>0</spring_reference>
+      <spring_stiffness>0</spring_stiffness>
+    </dynamics>
+    <use_parent_model_frame>1</use_parent_model_frame>
+  </axis>
 </joint>
 </gazebo>
