Commit message: Fixing manipulation stuff. Edited some CMakeLists.txt so they make sure arbie_msgs is built.

File: arbie_description/temp/arbie_temp.urdf (robot description, URDF)
Before this commit: robot arbie, 44 links, 43 joints
Joints:
- joint arm_2_joint: limit (none) -> lower=0.0 upper=3.14159265359 effort=1000.0 velocity=1; type continuous -> revolute
- joint arm_3_joint: limit (none) -> lower=0.0 upper=3.14159265359 effort=1000.0 velocity=1; type continuous -> revolute
- joint wrist_pitch_joint: limit (none) -> lower=1.57079632679 upper=-1.57079632679 effort=1000.0 velocity=1; type continuous -> revolute
- joint wrist_yaw_joint: limit (none) -> lower=1.57079632679 upper=-1.57079632679 effort=1000.0 velocity=1; type continuous -> revolute

Commit message: Added gripper joint control. Needed to update moveit package to include mimic joints in gripper group.

File: arbie_description/temp/arbie_temp.urdf (robot description, URDF)
Before this commit: robot arbie, 44 links, 43 joints
Joints:
- joint arm_1_joint: limit (none) -> effort=1000.0 velocity=1.5
- joint arm_2_joint: limit lower=0.0 upper=3.14159265359 effort=1000.0 velocity=1 -> lower=0.0 upper=3.14159265359 effort=1000.0 velocity=10
- joint arm_3_joint: limit lower=0.0 upper=3.14159265359 effort=1000.0 velocity=1 -> lower=0.0 upper=3.14159265359 effort=1000.0 velocity=10; origin xyz=-0.033 0.035 -0.45 rpy=0 0 0 -> xyz=-0.033 0.035 -0.45 rpy=-0.04 0 0
- joint wrist_pitch_joint: limit lower=1.57079632679 upper=-1.57079632679 effort=1000.0 velocity=1 -> lower=-1.57079632679 upper=1.57079632679 effort=1000.0 velocity=10
- joint wrist_roll_joint: limit (none) -> effort=1000.0 velocity=3.14159265359; origin xyz=0.0 0.019 0.0454 rpy=0 0 -1.5708 -> xyz=0.0 0.019 0.0454 rpy=0 0 0
- joint wrist_yaw_joint: limit lower=1.57079632679 upper=-1.57079632679 effort=1000.0 velocity=1 -> lower=-1.57079632679 upper=1.57079632679 effort=1000.0 velocity=10
